File: PCB/CawDrive.kicad_sch (KiCad schematic)
At the start: 67 parts, among them CN2 WAFER-SH1.0-6PWB, CN3 WAFER-SH1.0-4PWB, Q1 NMOS, U1 TJA1051T/3/1J, U10 WAFER-SH1.0-2PWB, U11 WAFER-SH1.0-2PWB, U12 WAFER-SH1.0-2PWB, U5 WAFER-SH1.0-2PWB, U6 WAFER-SH1.0-2PWB, U8 STM32F446RETx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

Commit message: refactor: 将符号表和封装导出到项目中
Parts:
- C1, C11, C12, C13, C14, C17, C18, C19, C2, C3, C4, C5, C6, C9: symbol Device:C_Small -> Library:C_Small
- CN2: symbol Rick_Connector:WAFER-SH1.0-6PWB -> Library:WAFER-SH1.0-6PWB
- CN3: symbol Rick_Connector:WAFER-SH1.0-4PWB -> Library:WAFER-SH1.0-4PWB
- D1, D2, D4, D6: symbol Device:LED_Small -> Library:LED_Small
- H1, H2, H3, H4, H8, H9: symbol Mechanical:MountingHole_Pad -> Library:MountingHole_Pad
- L1: symbol Device:L_Small -> Library:L_Small
- Q1: symbol Simulation_SPICE:NMOS -> Library:NMOS
- R1, R10, R11, R12, R15, R2, R20, R21, R22, R23, R24, R25, R26, R3, R4, R5, R6, R7, R8, R9: symbol Device:R_Small -> Library:R_Small
- TP1, TP2, TP3, TP4, TP5, TP6, TP7, TP8, TP9: symbol Connector:TestPoint -> Library:TestPoint
- TV1: symbol Rick_Diode:SMAJ36CA/TR13 -> Library:SMAJ36CA/TR13
- U1: symbol Rick_CAN:TJA1051T/3/1J -> Library:TJA1051T/3/1J
- U10, U11, U12, U5, U6: symbol Rick_Connector:WAFER-SH1.0-2PWB -> Library:WAFER-SH1.0-2PWB
- U8: symbol MCU_ST_STM32F4:STM32F446RETx -> Library:STM32F446RETx
- U9: symbol Rick_Sensor:MT6835GT-STD -> Library:MT6835GT-STD
- X1: symbol Rick_Device:Crystal_16MHz_15pF_3P -> Library:Crystal_16MHz_15pF_3P
