File: PCB/DRV8323RSRGZR.kicad_sch (KiCad schematic)
At the start: 42 parts, among them Q10 TPH3R704PL, Q11 TPH3R704PL, Q12 TPH3R704PL, Q7 TPH3R704PL, Q8 TPH3R704PL, Q9 TPH3R704PL, U2 TLV76733DRVR, U7 DRV8323RSRGZR

Commit message: refactor: 将符号表和封装导出到项目中
Parts:
- C10, C15, C16, C20, C21, C22, C23, C24, C25, C26, C27, C28, C29, C30, C31, C32, C33, C34, C35, C36, C37, C38, C7: symbol Device:C_Small -> Library:C_Small
- D3: symbol Device:D_Schottky_Small -> Library:D_Schottky_Small
- H5, H6, H7: symbol Mechanical:MountingHole_Pad -> Library:MountingHole_Pad
- L2: symbol Rick_Inductor:LQH5BPB220MT0L_22uH_±20%_1.4A -> Library:LQH5BPB220MT0L_22uH_±20%_1.4A
- Q10, Q11, Q12, Q7, Q8, Q9: symbol Rick_MOSFET:TPH3R704PL -> Library:TPH3R704PL
- R13, R14, R16, R17, R18, R19: symbol Device:R_Small -> Library:R_Small
- U2: symbol Rick_Regulator_Linear:TLV76733DRVR -> Library:TLV76733DRVR
- U7: symbol Rick_Drive:DRV8323RSRGZR -> Library:DRV8323RSRGZR
